File: motor_control.kicad_sch (KiCad schematic)
At the start: 12 parts, among them J3 Brushed DC Northeast, J4 Brushed DC Southeast, U1 STSPIN240

Commit message: Catalogued in raja.rocks
Parts:
- added C29, C31: 100nF, Capacitor_SMD:C_0201_0603Metric, symbol Device:C
- added C30: 10nF, Capacitor_SMD:C_0201_0603Metric, symbol Device:C
- added U5: MPU-9250, Sensor_Motion:InvenSense_QFN-24_3x3mm_P0.4mm, symbol Sensor_Motion:MPU-9250
Connections:
- net +3.3V: now also C30.2, C31.1, U5.1 (RESV_VDDIO), U5.13 (VDD), U5.8 (VDDIO)
- net GND: now also U1.1 (PHA), U1.15 (PHB), C29.2, C30.1, C31.2, U5.11 (FSYNC), U5.18 (GND), U5.20 (RESV_GND)
- net PA1: now reaches U1.16 (PWMB)
- net PA0: now reaches U1.2 (PWMA)
- new net: C29.1, U5.10 (REGOUT)
- new net MPU_CS: U5.22 (~{CS})
- new net SCLK: U5.23 (SCL/SCLK)
- new net SDI: U5.24 (SDA/MOSI)
- new net SDO: U5.9 (AD0/MISO)
- no-connect marks 0 -> 3
Other:
- moved on the sheet: C16, C17, C18, C20, J3, J4, R10, R6, R7, R8, R9, U1
