File: power.kicad_sch (KiCad schematic)
At the start: 20 parts, among them J1 JST_PH, J2 USB_C_Receptacle_PowerOnly_6P, U3 MCP1754S-3302xCB, U4 LTC4055

Commit message: Catalogued in raja.rocks
Parts:
- removed F1: 500mA, Fuse:Fuse_0402_1005Metric, symbol Device:Fuse
- removed R3, R4: 97.6k, Resistor_SMD:R_0201_0603Metric, symbol Device:R
- added F1: 500mA, Fuse:Fuse_1206_3216Metric, symbol Device:Polyfuse
- added RN1: 120k, Resistor_SMD:R_Array_Convex_4x1206, symbol Device:R_Pack04_Split
Connections:
- net -BATT: now also RN1.1 (R1.1), RN1.2 (R2.1)
- net at D2.1 (K): now also F1.1
- net at U4.11 (PROG): now also RN1.7 (R2.2)
- net at U4.9 (CLPROG): now also RN1.8 (R1.2)
- net at FB3.1: now also F1.2
- no-connect marks 4 -> 6
Other:
- moved on the sheet: D2
